File: IOB-generic.brd (EAGLE design)
At the start: 53.3 x 20.3 mm, 8 parts, among them J1 RJ12/6

Commit message: silkscreen and top fill, array
Parts:
- IOB: value CONNECTOR-IO4-IOBBARE -> CONNECTOR-IO4-IOBFULL
Other:
- board text added: "FID1"
- board text added: "FID2"
- board text added: "R10"
- board text added: "R11"
- board text added: "R12"
- board text added: "R9"
- board text added: "Yellow Soldermask White Silkscreen"
- board text removed: "Yellow Soldermask Black Silkscreen"
Changed lines of the file:
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@@
 <layer number="19" name="Unrouted" color="6" fill="1" visible="yes" active="yes"/>
 <layer number="20" name="Dimension" color="15" fill="1" visible="yes" active="yes"/>
-<layer number="21" name="tPlace" color="39" fill="1" visible="yes" active="yes"/>
-<layer number="22" name="bPlace" color="17" fill="1" visible="no" active="yes"/>
+<layer number="21" name="tPlace" color="8" fill="1" visible="yes" active="yes"/>
+<layer number="22" name="bPlace" color="8" fill="1" visible="no" active="yes"/>
 <layer number="23" name="tOrigins" color="30" fill="1" visible="yes" active="yes"/>
 <layer number="24" name="bOrigins" color="15" fill="1" visible="no" active="yes"/>
@@
 <layer number="60" name="bCarbon" color="7" fill="1" visible="no" active="no"/>
 <layer number="90" name="Modules" color="5" fill="1" visible="no" active="no"/>
-<layer number="100" name="Muster" color="7" fill="1" visible="no" active="no"/>
-<layer number="101" name="Hidden" color="57" fill="4" visible="yes" active="yes"/>
-<layer number="102" name="Changes" color="13" fill="1" visible="yes" active="yes"/>
-<layer number="103" name="tMap" color="29" fill="4" visible="yes" active="yes"/>
-<layer number="104" name="Name" color="16" fill="1" visible="yes" active="yes"/>
-<layer number="105" name="tPlate" color="7" fill="1" visible="yes" active="yes"/>
-<layer number="106" name="bPlate" color="7" fill="1" visible="yes" active="yes"/>
-<layer number="107" name="Crop" color="7" fill="1" visible="yes" active="yes"/>
-<layer number="108" name="fp8" color="7" fill="1" visible="yes" active="yes"/>
-<layer number="109" name="fp9" color="7" fill="1" visible="yes" active="yes"/>
-<layer number="110" name="fp0" color="7" fill="1" visible="yes" active="yes"/>
-<layer number="111" name="bdokum" color="7" fill="1" visible="yes" active="yes"/>
-<layer number="112" name="tSilk" color="7" fill="1" visible="no" active="no"/>
-<layer number="113" name="IDFDebug" color="7" fill="1" visible="yes" active="yes"/>
-<layer number="114" name="Rect_Pads" color="7" fill="1" visible="yes" active="yes"/>
-<layer number="115" name="_tsilk" color="7" fill="1" visible="yes" active="yes"/>
-<layer number="116" name="Patch_BOT" color="9" fill="4" visible="yes" active="yes"/>
-<layer number="117" name="tTestmark" color="7" fill="1" visible="yes" active="yes"/>
-<layer number="118" name="Rect_Pads" color="7" fill="1" visible="no" active="no"/>
-<layer number="119" name="_tNames" color="7" fill="1" visible="yes" active="yes"/>
-<layer number="120" name="_bNames" color="7" fill="1" visible="yes" active="yes"/>
-<layer number="121" name="_tsilk" color="7" fill="1" visible="yes" active="yes"/>
-<layer number="122" name="_bsilk" color="7" fill="1" visible="yes" active="yes"/>
-<layer number="123" name="tTestmark" color="7" fill="1" visible="yes" active="yes"/>
-<layer number="124" name="bTestmark" color="7" fill="1" visible="yes" active="yes"/>
-<layer number="125" name="_tNames" color="7" fill="1" visible="yes" active="yes"/>
-<layer number="126" name="_bNames" color="7" fill="1" visible="yes" active="yes"/>
-<layer number="127" name="_tValues" color="7" fill="1" visible="no" active="no"/>
-<layer number="128" name="_bValues" color="7" fill="1" visible="no" active="no"/>
-<layer number="129" name="Mask" color="7" fill="1" visible="yes" active="yes"/>
-<layer number="130" name="SMDSTROOK" color="7" fill="1" visible="yes" active="yes"/>
-<layer number="131" name="tAdjust" color="7" fill="1" visible="yes" active="yes"/>
-<layer number="132" name="bAdjust" color="7" fill="1" visible="yes" active="yes"/>
-<layer number="144" name="Drill_legend" color="7" fill="1" visible="yes" active="yes"/>
-<layer number="146" name="Housing" color="7" fill="1" visible="yes" active="yes"/>
-<layer number="147" name="Edge" color="7" fill="1" visible="yes" active="yes"/>
-<layer number="148" name="ReferenceLC" color="7" fill="1" visible="yes" active="yes"/>
-<layer number="149" name="ReferenceLS" color="7" fill="1" visible="yes" active="yes"/>
-<layer number="150" name="Notes" color="7" fill="1" visible="yes" active="yes"/>
-<layer number="151" name="HeatSink" color="7" fill="1" visible="yes" active="yes"/>
-<layer number="152" name="_bDocu" color="7" fill="1" visible="no" active="no"/>
-<layer number="153" name="FabDoc1" color="7" fill="1" visible="yes" active="yes"/>
-<layer number="154" name="FabDoc2" color="7" fill="1" visible="yes" active="yes"/>
-<layer number="155" name="FabDoc3" color="7" fill="1" visible="yes" active="yes"/>
-<layer number="199" name="Contour" color="7" fill="1" visible="yes" active="yes"/>
-<layer number="200" name="200bmp" color="1" fill="10" visible="yes" active="yes"/>
-<layer number="201" name="201bmp" color="2" fill="10" visible="yes" active="yes"/>
-<layer number="202" name="202bmp" color="3" fill="10" visible="yes" active="yes"/>
-<layer number="203" name="203bmp" color="4" fill="10" visible="yes" active="yes"/>
-<layer number="204" name="204bmp" color="5" fill="10" visible="yes" active="yes"/>
-<layer number="205" name="205bmp" color="6" fill="10" visible="yes" active="yes"/>
-<layer number="206" name="206bmp" color="7" fill="10" visible="yes" active="yes"/>
-<layer number="207" name="207bmp" color="8" fill="10" visible="yes" active="yes"/>
-<layer number="208" name="208bmp" color="9" fill="10" visible="yes" active="yes"/>
-<layer number="209" name="209bmp" color="7" fill="1" visible="yes" active="yes"/>
-<layer number="210" name="210bmp" color="7" fill="1" visible="yes" active="yes"/>
-<layer number="211" name="211bmp" color="12" fill="1" visible="no" active="no"/>
-<layer number="212" name="212bmp" color="13" fill="1" visible="no" active="no"/>
-<layer number="213" name="213bmp" color="14" fill="1" visible="no" active="no"/>
-<layer number="214" name="214bmp" color="15" fill="1" visible="no" active="no"/>
-<layer number="215" name="215bmp" color="16" fill="1" visible="no" active="no"/>
-<layer number="216" name="216bmp" color="17" fill="1" visible="no" active="no"/>
-<layer number="217" name="217bmp" color="18" fill="1" visible="no" active="no"/>
-<layer number="218" name="218bmp" color="19" fill="1" visible="no" active="no"/>
-<layer number="219" name="219bmp" color="20" fill="1" visible="no" active="no"/>
-<layer number="220" name="220bmp" color="21" fill="1" visible="no" active="no"/>
-<layer number="221" name="221bmp" color="22" fill="1" visible="no" active="no"/>
-<layer number="222" name="222bmp" color="23" fill="1" visible="no" active="no"/>
-<layer number="223" name="223bmp" color="24" fill="1" visible="no" active="no"/>
-<layer number="224" name="224bmp" color="25" fill="1" visible="no" active="no"/>
-<layer number="225" name="225bmp" color="7" fill="1" visible="yes" active="yes"/>
-<layer number="226" name="226bmp" color="7" fill="1" visible="yes" active="yes"/>
-<layer number="227" name="227bmp" color="7" fill="1" visible="yes" active="yes"/>
-<layer number="228" name="228bmp" color="7" fill="1" visible="yes" active="yes"/>
-<layer number="229" name="229bmp" color="7" fill="1" visible="yes" active="yes"/>
-<layer number="230" name="230bmp" color="7" fill="1" visible="yes" active="yes"/>
-<layer number="231" name="231bmp" color="7" fill="1" visible="yes" active="yes"/>
-<layer number="232" name="Eagle3D_PG2" color="7" fill="1" visible="yes" active="yes"/>
-<layer number="233" name="Eagle3D_PG3" color="7" fill="1" visible="yes" active="yes"/>
-<layer number="247" name="wrappinf" color="7" fill="1" visible="yes" active="yes"/>
-<layer number="248" name="Housing" color="7" fill="1" visible="no" active="no"/>
-<layer number="249" name="Edge" color="7" fill="1" visible="no" active="no"/>
-<layer number="250" name="Descript" color="3" fill="1" visible="no" active="no"/>
-<layer number="251" name="SMDround" color="12" fill="11" visible="no" active="no"/>
-<layer number="252" name="BR-BS" color="7" fill="1" visible="yes" active="yes"/>
-<layer number="253" name="BR-LS" color="7" fill="1" visible="yes" active="yes"/>
-<layer number="254" name="cooling" color="7" fill="1" visible="yes" active="yes"/>
-<layer number="255" name="routoute" color="7" fill="1" visible="yes" active="yes"/>
+<layer number="125" name="_tNames" color="14" fill="1" visible="yes" active="yes"/>
 </layers>
 <board>
@@
 <text x="15.875" y="4.064" size="1.778" layer="22" font="vector" rot="MR180">Generic Quad I/O</text>
 <text x="-3.81" y="1.905" size="1.27" layer="48" font="vector" ratio="10" rot="R90">Yellow Soldermask
-Black Silkscreen</text>
+White Silkscreen</text>
 <text x="31.496" y="13.716" size="0.8128" layer="21" font="vector" ratio="10" rot="SR90"> Cut if
 &lt; using
@@
 <text x="4.699" y="5.969" size="1.016" layer="21" font="vector" rot="R90">2020.03</text>
 <text x="55.245" y="1.27" size="1.4224" layer="48" font="vector" ratio="10" rot="R90">Yellow Headers</text>
+<text x="-5.08" y="0.127" size="1.016" layer="125" font="vector">FID1</text>
+<text x="53.975" y="18.923" size="1.016" layer="125" font="vector">FID2</text>
+<text x="32.258" y="11.4935" size="0.4064" layer="125" font="vector" rot="R180">R9</text>
+<text x="32.258" y="8.9535" size="0.4064" layer="125" font="vector" rot="R180">R10</text>
+<text x="32.258" y="6.2865" size="0.4064" layer="125" font="vector" rot="R180">R11</text>
+<text x="32.131" y="3.3655" size="0.4064" layer="125" font="vector" rot="R180">R12</text>
 </plain>
 <attributes>
@@
 <attribute name="VALUE" x="-0.889" y="5.842" size="1.016" layer="27" font="vector" rot="R90"/>
 </element>
-<element name="IOB" library="SPCoast" package="IO4-IOB" value="CONNECTOR-IO4-IOBBARE" x="0" y="0"/>
+<element name="IOB" library="SPCoast" package="IO4-IOB" value="CONNECTOR-IO4-IOBFULL" x="0" y="0"/>
 <element name="R9" library="SPCoast" package="AXIAL-0.4-RES" value="NOSTUFF" x="30.734" y="12.446" smashed="yes" rot="R180">
 <attribute name="NAME" x="32.258" y="11.4935" size="0.4064" layer="25" font="vector" rot="R180"/>

Commit message: Fab Date, DRC
Routing:
- net !IO4: vias 1 -> 0
- net !IO3: vias 1 -> 0
- net !IO2: vias 1 -> 0
- net !IO1: vias 1 -> 0
Other:
- board text added: "2020.08"
- board text removed: "2020.03"
Changed lines of the file:
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@@
 &lt; using
 resistor</text>
-<text x="4.699" y="5.969" size="1.016" layer="21" font="vector" rot="R90">2020.03</text>
+<text x="4.699" y="5.969" size="1.016" layer="21" font="vector" rot="R90">2020.08</text>
 <text x="55.245" y="1.27" size="1.4224" layer="48" font="vector" ratio="10" rot="R90">Yellow Headers</text>
 <text x="-5.08" y="0.127" size="1.016" layer="125" font="vector">FID1</text>
@@
 <contactref element="J1" pad="2@1"/>
 <wire x1="25.654" y1="12.446" x2="11.303" y2="12.446" width="0.4064" layer="16"/>
-<wire x1="11.303" y1="12.446" x2="11.176" y2="12.573" width="0.4064" layer="1"/>
+<wire x1="11.303" y1="12.446" x2="11.176" y2="12.573" width="0.4064" layer="16"/>
 <wire x1="6.096" y1="7.239" x2="4.572" y2="7.239" width="0.3048" layer="1"/>
 <wire x1="4.572" y1="7.239" x2="4.318" y2="7.493" width="0.3048" layer="1"/>
@@
 <wire x1="4.318" y1="11.176" x2="5.715" y2="12.573" width="0.3048" layer="1"/>
 <wire x1="5.715" y1="12.573" x2="11.176" y2="12.573" width="0.3048" layer="1"/>
-<via x="11.303" y="12.446" extent="1-16" drill="0.6"/>
 </signal>
 <signal name="!IO2" class="2">
@@
 <contactref element="J1" pad="3@1"/>
 <wire x1="25.654" y1="9.906" x2="11.557" y2="9.906" width="0.4064" layer="16"/>
-<wire x1="11.557" y1="9.906" x2="11.43" y2="10.033" width="0.4064" layer="1"/>
+<wire x1="11.557" y1="9.906" x2="11.43" y2="10.033" width="0.4064" layer="16"/>
 <wire x1="7.874" y1="8.255" x2="9.144" y2="8.255" width="0.254" layer="16"/>
 <wire x1="9.144" y1="8.255" x2="9.398" y2="8.509" width="0.254" layer="16"/>
@@
 <wire x1="9.398" y1="9.779" x2="9.652" y2="10.033" width="0.254" layer="16"/>
 <wire x1="9.652" y1="10.033" x2="11.43" y2="10.033" width="0.254" layer="16"/>
-<via x="11.557" y="9.906" extent="1-16" drill="0.6"/>
 </signal>
 <signal name="!IO3" class="2">
@@
 <contactref element="J1" pad="4@1"/>
 <wire x1="25.654" y1="7.366" x2="11.303" y2="7.366" width="0.4064" layer="16"/>
-<wire x1="11.303" y1="7.366" x2="11.176" y2="7.493" width="0.4064" layer="1"/>
+<wire x1="11.303" y1="7.366" x2="11.176" y2="7.493" width="0.4064" layer="16"/>
 <wire x1="6.096" y1="9.271" x2="4.826" y2="9.271" width="0.254" layer="16"/>
 <wire x1="4.826" y1="9.271" x2="4.699" y2="9.144" width="0.254" layer="16"/>
@@
 <wire x1="9.017" y1="7.112" x2="9.398" y2="7.493" width="0.254" layer="16"/>
 <wire x1="9.398" y1="7.493" x2="11.176" y2="7.493" width="0.254" layer="16"/>
-<via x="11.303" y="7.366" extent="1-16" drill="0.6"/>
 </signal>
 <signal name="!IO4" class="2">
@@
 <contactref element="J1" pad="5@1"/>
 <wire x1="25.654" y1="4.826" x2="11.557" y2="4.826" width="0.4064" layer="16"/>
-<wire x1="11.557" y1="4.826" x2="11.43" y2="4.953" width="0.4064" layer="1"/>
+<wire x1="11.557" y1="4.826" x2="11.43" y2="4.953" width="0.4064" layer="16"/>
 <wire x1="7.874" y1="10.287" x2="9.144" y2="10.287" width="0.254" layer="1"/>
 <wire x1="9.144" y1="10.287" x2="9.398" y2="10.033" width="0.254" layer="1"/>
@@
 <wire x1="9.398" y1="5.207" x2="9.652" y2="4.953" width="0.254" layer="1"/>
 <wire x1="9.652" y1="4.953" x2="11.43" y2="4.953" width="0.254" layer="1"/>
-<via x="11.557" y="4.826" extent="1-16" drill="0.6"/>
 </signal>
 <signal name="VOUT" class="1">
